File: hardware/psu.sch (KiCad schematic (older format))
At the start: 14 parts

Commit message: Add user IO, programming headers
Parts:
- added BT1: Battery, symbol Battery
- gave numbers to parts that had none: 13
Connections:
- net GNDD: now also BT1.2
- new net BATTERY+: BT1.1
Other:
- moved on the sheet: 15k1, 18k1, C10, C12, D4, U2
