File: hardware/analog.sch (KiCad schematic (older format))
At the start: 23 parts, among them U3 LTC6257

Commit message: Start placement of parts
Parts:
- C14, C15, C16, C17, C18: footprint (none) -> footprints:SMD0805-CAP-M
- C19, C20, C21: footprint (none) -> footprints:C_Radial_D6.3_L13_P2-5_Bent
- R10, R11, R12, R13, R14, R15, R16, R17, R18, R19, R20, R21, R22, R9: footprint (none) -> footprints:SMD0805-RES-M
- U3: footprint (none) -> footprints:MSOP16-05mm-M
Changed lines of the file:
@@
 F 0 "U3" H 3300 3600 60  0000 C CNN
 F 1 "LTC6257" H 3400 3200 50  0000 C CNN
-F 2 "" H 3250 3400 60  0000 C CNN
+F 2 "footprints:MSOP16-05mm-M" H 3250 3400 60  0001 C CNN
 F 3 "" H 3250 3400 60  0000 C CNN
 	2    3250 3400
@@
 F 0 "U3" H 3250 1850 60  0000 C CNN
 F 1 "LTC6257" H 3350 1450 50  0000 C CNN
-F 2 "" H 3200 1650 60  0000 C CNN
+F 2 "footprints:MSOP16-05mm-M" H 3200 1650 60  0001 C CNN
 F 3 "" H 3200 1650 60  0000 C CNN
 	1    3200 1650
@@
 F 0 "R20" V 3230 3950 50  0000 C CNN
 F 1 "10k 1%" V 3050 3950 50  0000 C CNN
-F 2 "" V 3080 3950 50  0000 C CNN
+F 2 "footprints:SMD0805-RES-M" V 3080 3950 50  0001 C CNN
 F 3 "" H 3150 3950 50  0000 C CNN
 	1    3150 3950
@@
 F 0 "R11" V 2380 3300 50  0000 C CNN
 F 1 "10k 1%" V 2200 3300 50  0000 C CNN
-F 2 "" V 2230 3300 50  0000 C CNN
+F 2 "footprints:SMD0805-RES-M" V 2230 3300 50  0001 C CNN
 F 3 "" H 2300 3300 50  0000 C CNN
 	1    2300 3300
@@
 F 0 "R12" V 2380 3500 50  0000 C CNN
 F 1 "10k  1%" V 2450 3500 50  0000 C CNN
-F 2 "" V 2230 3500 50  0000 C CNN
+F 2 "footprints:SMD0805-RES-M" V 2230 3500 50  0001 C CNN
 F 3 "" H 2300 3500 50  0000 C CNN
 	1    2300 3500
@@
 F 0 "R18" V 2680 3000 50  0000 C CNN
 F 1 "10k 1%" V 2500 3000 50  0000 C CNN
-F 2 "" V 2530 3000 50  0000 C CNN
+F 2 "footprints:SMD0805-RES-M" V 2530 3000 50  0001 C CNN
 F 3 "" H 2600 3000 50  0000 C CNN
 	1    2600 3000
@@
 $EndComp
 $Comp
-L VCOM #PWR39
+L VCOM #PWR035
 U 1 1 57387E0B
 P 2600 2750
-F 0 "#PWR39" H 2600 2600 50  0001 C CNN
+F 0 "#PWR035" H 2600 2600 50  0001 C CNN
 F 1 "VCOM" H 2600 2900 50  0000 C CNN
 F 2 "" H 2600 2750 50  0000 C CNN
@@
 F 0 "U3" H 3450 5300 60  0000 C CNN
 F 1 "LTC6257" H 3550 4900 50  0000 C CNN
-F 2 "" H 3400 5100 60  0000 C CNN
+F 2 "footprints:MSOP16-05mm-M" H 3400 5100 60  0001 C CNN
 F 3 "" H 3400 5100 60  0000 C CNN
 	3    3400 5100
@@
 F 0 "R21" V 3380 5650 50  0000 C CNN
 F 1 "10k 1%" V 3200 5650 50  0000 C CNN
-F 2 "" V 3230 5650 50  0000 C CNN
+F 2 "footprints:SMD0805-RES-M" V 3230 5650 50  0001 C CNN
 F 3 "" H 3300 5650 50  0000 C CNN
 	1    3300 5650
@@
 F 0 "R13" V 2530 5000 50  0000 C CNN
 F 1 "10k 1%" V 2350 5000 50  0000 C CNN
-F 2 "" V 2380 5000 50  0000 C CNN
+F 2 "footprints:SMD0805-RES-M" V 2380 5000 50  0001 C CNN
 F 3 "" H 2450 5000 50  0000 C CNN
 	1    2450 5000
@@
 F 0 "R14" V 2530 5200 50  0000 C CNN
 F 1 "10k 1%" V 2600 5200 50  0000 C CNN
-F 2 "" V 2380 5200 50  0000 C CNN
+F 2 "footprints:SMD0805-RES-M" V 2380 5200 50  0001 C CNN
 F 3 "" H 2450 5200 50  0000 C CNN
 	1    2450 5200
@@
 F 0 "R19" V 2830 4700 50  0000 C CNN
 F 1 "10k 1%" V 2650 4700 50  0000 C CNN
-F 2 "" V 2680 4700 50  0000 C CNN
+F 2 "footprints:SMD0805-RES-M" V 2680 4700 50  0001 C CNN
 F 3 "" H 2750 4700 50  0000 C CNN
 	1    2750 4700
@@
 $EndComp
 $Comp
-L VCOM #PWR40
+L VCOM #PWR036
 U 1 1 57388860
 P 2750 4450
-F 0 "#PWR40" H 2750 4300 50  0001 C CNN
+F 0 "#PWR036" H 2750 4300 50  0001 C CNN
 F 1 "VCOM" H 2750 4600 50  0000 C CNN
 F 2 "" H 2750 4450 50  0000 C CNN
@@
 F 0 "R9" V 2080 1200 50  0000 C CNN
 F 1 "1meg" V 1900 1200 50  0000 C CNN
-F 2 "" V 1930 1200 50  0000 C CNN
+F 2 "footprints:SMD0805-RES-M" V 1930 1200 50  0001 C CNN
 F 3 "" H 2000 1200 50  0000 C CNN
 	1    2000 1200
@@
 F 0 "R10" V 2080 1800 50  0000 C CNN
 F 1 "1meg" V 1900 1800 50  0000 C CNN
-F 2 "" V 1930 1800 50  0000 C CNN
+F 2 "footprints:SMD0805-RES-M" V 1930 1800 50  0001 C CNN
 F 3 "" H 2000 1800 50  0000 C CNN
 	1    2000 1800
@@
 F 0 "C14" H 2275 1900 50  0000 L CNN
 F 1 "2u2" H 2275 1700 50  0000 L CNN
-F 2 "" H 2288 1650 50  0000 C CNN
+F 2 "footprints:SMD0805-CAP-M" H 2288 1650 50  0001 C CNN
 F 3 "" H 2250 1800 50  0000 C CNN
 	1    2250 1800
@@
 $EndComp
 $Comp
-L VAA #PWR35
+L VAA #PWR037
 U 1 1 57389681
 P 2000 950
-F 0 "#PWR35" H 2000 800 50  0001 C CNN
+F 0 "#PWR037" H 2000 800 50  0001 C CNN
 F 1 "VAA" H 2000 1100 50  0000 C CNN
 F 2 "" H 2000 950 50  0000 C CNN
@@
 $EndComp
 $Comp
-L GNDA #PWR37
+L GNDA #PWR038
 U 1 1 573898FE
 P 2250 2100
-F 0 "#PWR37" H 2250 1850 50  0001 C CNN
+F 0 "#PWR038" H 2250 1850 50  0001 C CNN
 F 1 "GNDA" H 2250 1950 50  0000 C CNN
 F 2 "" H 2250 2100 50  0000 C CNN
@@
 $EndComp
 $Comp
-L GNDA #PWR36
+L GNDA #PWR039
 U 1 1 5738993C
 P 2000 2100
-F 0 "#PWR36" H 2000 1850 50  0001 C CNN
+F 0 "#PWR039" H 2000 1850 50  0001 C CNN
 F 1 "GNDA" H 2000 1950 50  0000 C CNN
 F 2 "" H 2000 2100 50  0000 C CNN
@@
 $EndComp
 $Comp
-L GNDA #PWR42
+L GNDA #PWR040
 U 1 1 573899E3
 P 3100 2100
-F 0 "#PWR42" H 3100 1850 50  0001 C CNN
+F 0 "#PWR040" H 3100 1850 50  0001 C CNN
 F 1 "GNDA" H 3100 1950 50  0000 C CNN
 F 2 "" H 3100 2100 50  0000 C CNN
@@
 $EndComp
 $Comp
-L VAA #PWR41
+L VAA #PWR041
 U 1 1 5738A097
 P 3100 950
-F 0 "#PWR41" H 3100 800 50  0001 C CNN
+F 0 "#PWR041" H 3100 800 50  0001 C CNN
 F 1 "VAA" H 3100 1100 50  0000 C CNN
 F 2 "" H 3100 950 50  0000 C CNN
@@
 $EndComp
 $Comp
-L VCOM #PWR44
+L VCOM #PWR042
 U 1 1 5738A7C9
 P 3900 1600
-F 0 "#PWR44" H 3900 1450 50  0001 C CNN
+F 0 "#PWR042" H 3900 1450 50  0001 C CNN
 F 1 "VCOM" H 3900 1750 50  0000 C CNN
 F 2 "" H 3900 1600 50  0000 C CNN
@@
 F 0 "C18" H 3425 1150 50  0000 L CNN
 F 1 "2u2" H 3425 950 50  0000 L CNN
-F 2 "" H 3438 900 50  0000 C CNN
+F 2 "footprints:SMD0805-CAP-M" H 3438 900 50  0001 C CNN
 F 3 "" H 3400 1050 50  0000 C CNN
 	1    3400 1050
@@
 $EndComp
 $Comp
-L GNDA #PWR43
+L GNDA #PWR043
 U 1 1 5738B8B9
 P 3600 1150
-F 0 "#PWR43" H 3600 900 50  0001 C CNN
+F 0 "#PWR043" H 3600 900 50  0001 C CNN
 F 1 "GNDA" H 3600 1000 50  0000 C CNN
 F 2 "" H 3600 1150 50  0000 C CNN
@@
 F 0 "C19" H 4175 3500 50  0000 L CNN
 F 1 "470u" H 4175 3300 50  0000 L CNN
-F 2 "" H 4188 3250 50  0000 C CNN
+F 2 "footprints:C_Radial_D6.3_L13_P2-5_Bent" H 4188 3250 50  0001 C CNN
 F 3 "" H 4150 3400 50  0000 C CNN
 	1    4150 3400
@@
 F 0 "C21" H 4225 6800 50  0000 L CNN
 F 1 "470u" H 4225 6600 50  0000 L CNN
-F 2 "" H 4238 6550 50  0000 C CNN
+F 2 "footprints:C_Radial_D6.3_L13_P2-5_Bent" H 4238 6550 50  0001 C CNN
 F 3 "" H 4200 6700 50  0000 C CNN
 	1    4200 6700
@@
 F 0 "U3" H 3450 6900 60  0000 C CNN
 F 1 "LTC6257" H 3550 6500 50  0000 C CNN
-F 2 "" H 3400 6700 60  0000 C CNN
+F 2 "footprints:MSOP16-05mm-M" H 3400 6700 60  0001 C CNN
 F 3 "" H 3400 6700 60  0000 C CNN
 	4    3400 6700
@@
 F 0 "R15" V 2530 6400 50  0000 C CNN
 F 1 "10k" V 2450 6400 50  0000 C CNN
-F 2 "" V 2380 6400 50  0000 C CNN
+F 2 "footprints:SMD0805-RES-M" V 2380 6400 50  0001 C CNN
 F 3 "" H 2450 6400 50  0000 C CNN
 	1    2450 6400
@@
 F 0 "R16" V 2530 6600 50  0000 C CNN
 F 1 "10k" V 2450 6600 50  0000 C CNN
-F 2 "" V 2380 6600 50  0000 C CNN
+F 2 "footprints:SMD0805-RES-M" V 2380 6600 50  0001 C CNN
 F 3 "" H 2450 6600 50  0000 C CNN
 	1    2450 6600
@@
 F 0 "R17" V 2530 6900 50  0000 C CNN
 F 1 "10k" V 2450 6900 50  0000 C CNN
-F 2 "" V 2380 6900 50  0000 C CNN
+F 2 "footprints:SMD0805-RES-M" V 2380 6900 50  0001 C CNN
 F 3 "" H 2450 6900 50  0000 C CNN
 	1    2450 6900
@@
 F 0 "R22" V 3380 7200 50  0000 C CNN
 F 1 "10k" V 3300 7200 50  0000 C CNN
-F 2 "" V 3230 7200 50  0000 C CNN
+F 2 "footprints:SMD0805-RES-M" V 3230 7200 50  0001 C CNN
 F 3 "" H 3300 7200 50  0000 C CNN
 	1    3300 7200
@@
 	1850 6600 2300 6600
 $Comp
-L VCOM #PWR38
+L VCOM #PWR044
 U 1 1 573B619B
 P 2250 6850
-F 0 "#PWR38" H 2250 6700 50  0001 C CNN
+F 0 "#PWR044" H 2250 6700 50  0001 C CNN
 F 1 "VCOM" H 2250 7000 50  0000 C CNN
 F 2 "" H 2250 6850 50  0000 C CNN
@@
 F 0 "C20" H 4225 5200 50  0000 L CNN
 F 1 "470u" H 4225 5000 50  0000 L CNN
-F 2 "" H 4238 4950 50  0000 C CNN
+F 2 "footprints:C_Radial_D6.3_L13_P2-5_Bent" H 4238 4950 50  0001 C CNN
 F 3 "" H 4200 5100 50  0000 C CNN
 	1    4200 5100
@@
 F 0 "C15" H 3175 4250 50  0000 L CNN
 F 1 "TBD" H 3175 4050 50  0000 L CNN
-F 2 "" H 3188 4000 50  0000 C CNN
+F 2 "footprints:SMD0805-CAP-M" H 3188 4000 50  0001 C CNN
 F 3 "" H 3150 4150 50  0000 C CNN
 	1    3150 4150
@@
 F 0 "C16" H 3325 5950 50  0000 L CNN
 F 1 "C" H 3325 5750 50  0000 L CNN
-F 2 "" H 3338 5700 50  0000 C CNN
+F 2 "footprints:SMD0805-CAP-M" H 3338 5700 50  0001 C CNN
 F 3 "" H 3300 5850 50  0000 C CNN
 	1    3300 5850
@@
 F 0 "C17" H 3325 7600 50  0000 L CNN
 F 1 "TBD" H 3325 7400 50  0000 L CNN
-F 2 "" H 3338 7350 50  0000 C CNN
+F 2 "footprints:SMD0805-CAP-M" H 3338 7350 50  0001 C CNN
 F 3 "" H 3300 7500 50  0000 C CNN
 	1    3300 7500

Commit message: Fix #9
Connections:
- net LEFT_OUT: no longer R15.2
- net RIGHT_OUT: no longer R16.2
- net LEFT_SE: now reaches C15.1, C19.2, R20.1, U3.7
- net LEFT_SE: now also R15.2
- net RIGHT_SE: now reaches C16.1, C20.2, R21.1, U3.10
- net RIGHT_SE: now also R16.2
Changed lines of the file:
@@
 Text HLabel 1850 5200 0    60   Input ~ 0
 N_RIGHT
-Text HLabel 1850 6400 0    60   Input ~ 0
-LEFT_OUT
-Text HLabel 1850 6600 0    60   Input ~ 0
-RIGHT_OUT
 Text HLabel 4850 5100 2    60   Output ~ 0
 RIGHT_OUT
@@
 	1900 2050 2000 2050
 Connection ~ 2000 2050
+Text Label 3550 5650 0    60   ~ 0
+RIGHT_SE
+Text Label 3500 3950 0    60   ~ 0
+LEFT_SE
+Text Label 1850 6400 2    60   ~ 0
+LEFT_SE
+Text Label 1850 6600 2    60   ~ 0
+RIGHT_SE
 $EndSCHEMATC

Commit message: Fix #8
Connections:
- net LEFT_OPAMP+: now reaches R11.1, R18.1, U3.5 (+)
- net LEFT_OPAMP-: now reaches C15.2, R12.1, R20.2, U3.6 (-)
- net RIGHT_OPAMP-: now reaches C16.2, R14.1, R21.2, U3.11 (-)
- net RIGHT_OPAMP+: now reaches R13.1, R19.1, U3.12 (+)
- net N_LEFT renamed LO_N
- net N_RIGHT renamed RO_N
- net P_LEFT renamed LO_P
- net P_RIGHT renamed RO_P
Other:
- moved on the sheet: R11, R12, R13, R14
Changed lines of the file:
@@
 L R R11
 U 1 1 57387AB6
-P 2300 3300
-F 0 "R11" V 2380 3300 50  0000 C CNN
-F 1 "10k 1%" V 2200 3300 50  0000 C CNN
-F 2 "footprints:SMD0805-RES-M" V 2230 3300 50  0001 C CNN
-F 3 "" H 2300 3300 50  0000 C CNN
-	1    2300 3300
+P 1450 3300
+F 0 "R11" V 1530 3300 50  0000 C CNN
+F 1 "10k 1%" V 1350 3300 50  0000 C CNN
+F 2 "footprints:SMD0805-RES-M" V 1380 3300 50  0001 C CNN
+F 3 "" H 1450 3300 50  0000 C CNN
+	1    1450 3300
 	0    1    1    0
 $EndComp
@@
 L R R12
 U 1 1 57387B69
-P 2300 3500
-F 0 "R12" V 2380 3500 50  0000 C CNN
-F 1 "10k  1%" V 2450 3500 50  0000 C CNN
-F 2 "footprints:SMD0805-RES-M" V 2230 3500 50  0001 C CNN
-F 3 "" H 2300 3500 50  0000 C CNN
-	1    2300 3500
+P 1450 3500
+F 0 "R12" V 1530 3500 50  0000 C CNN
+F 1 "10k  1%" V 1600 3500 50  0000 C CNN
+F 2 "footprints:SMD0805-RES-M" V 1380 3500 50  0001 C CNN
+F 3 "" H 1450 3500 50  0000 C CNN
+	1    1450 3500
 	0    1    1    0
 $EndComp
@@
 $EndComp
 $Comp
-L VCOM #PWR035
+L VCOM #PWR037
 U 1 1 57387E0B
 P 2600 2750
-F 0 "#PWR035" H 2600 2600 50  0001 C CNN
+F 0 "#PWR037" H 2600 2600 50  0001 C CNN
 F 1 "VCOM" H 2600 2900 50  0000 C CNN
 F 2 "" H 2600 2750 50  0000 C CNN
@@
 L R R13
 U 1 1 57388842
-P 2450 5000
-F 0 "R13" V 2530 5000 50  0000 C CNN
-F 1 "10k 1%" V 2350 5000 50  0000 C CNN
-F 2 "footprints:SMD0805-RES-M" V 2380 5000 50  0001 C CNN
-F 3 "" H 2450 5000 50  0000 C CNN
-	1    2450 5000
+P 1600 5000
+F 0 "R13" V 1680 5000 50  0000 C CNN
+F 1 "10k 1%" V 1500 5000 50  0000 C CNN
+F 2 "footprints:SMD0805-RES-M" V 1530 5000 50  0001 C CNN
+F 3 "" H 1600 5000 50  0000 C CNN
+	1    1600 5000
 	0    1    1    0
 $EndComp
@@
 L R R14
 U 1 1 57388848
-P 2450 5200
-F 0 "R14" V 2530 5200 50  0000 C CNN
-F 1 "10k 1%" V 2600 5200 50  0000 C CNN
-F 2 "footprints:SMD0805-RES-M" V 2380 5200 50  0001 C CNN
-F 3 "" H 2450 5200 50  0000 C CNN
-	1    2450 5200
+P 1600 5200
+F 0 "R14" V 1680 5200 50  0000 C CNN
+F 1 "10k 1%" V 1750 5200 50  0000 C CNN
+F 2 "footprints:SMD0805-RES-M" V 1530 5200 50  0001 C CNN
+F 3 "" H 1600 5200 50  0000 C CNN
+	1    1600 5200
 	0    1    1    0
 $EndComp
@@
 $EndComp
 $Comp
-L VCOM #PWR036
+L VCOM #PWR038
 U 1 1 57388860
 P 2750 4450
-F 0 "#PWR036" H 2750 4300 50  0001 C CNN
+F 0 "#PWR038" H 2750 4300 50  0001 C CNN
 F 1 "VCOM" H 2750 4600 50  0000 C CNN
 F 2 "" H 2750 4450 50  0000 C CNN
@@
 $EndComp
 $Comp
-L VAA #PWR037
+L VAA #PWR039
 U 1 1 57389681
 P 2000 950
-F 0 "#PWR037" H 2000 800 50  0001 C CNN
+F 0 "#PWR039" H 2000 800 50  0001 C CNN
 F 1 "VAA" H 2000 1100 50  0000 C CNN
 F 2 "" H 2000 950 50  0000 C CNN
@@
 $EndComp
 $Comp
-L GNDA #PWR038
+L GNDA #PWR040
 U 1 1 573898FE
 P 2250 2100
-F 0 "#PWR038" H 2250 1850 50  0001 C CNN
+F 0 "#PWR040" H 2250 1850 50  0001 C CNN
 F 1 "GNDA" H 2250 1950 50  0000 C CNN
 F 2 "" H 2250 2100 50  0000 C CNN
@@
 $EndComp
 $Comp
-L GNDA #PWR039
+L GNDA #PWR041
 U 1 1 5738993C
 P 2000 2100
-F 0 "#PWR039" H 2000 1850 50  0001 C CNN
+F 0 "#PWR041" H 2000 1850 50  0001 C CNN
 F 1 "GNDA" H 2000 1950 50  0000 C CNN
 F 2 "" H 2000 2100 50  0000 C CNN
@@
 $EndComp
 $Comp
-L GNDA #PWR040
+L GNDA #PWR042
 U 1 1 573899E3
 P 3100 2100
-F 0 "#PWR040" H 3100 1850 50  0001 C CNN
+F 0 "#PWR042" H 3100 1850 50  0001 C CNN
 F 1 "GNDA" H 3100 1950 50  0000 C CNN
 F 2 "" H 3100 2100 50  0000 C CNN
@@
 $EndComp
 $Comp
-L VAA #PWR041
+L VAA #PWR043
 U 1 1 5738A097
 P 3100 950
-F 0 "#PWR041" H 3100 800 50  0001 C CNN
+F 0 "#PWR043" H 3100 800 50  0001 C CNN
 F 1 "VAA" H 3100 1100 50  0000 C CNN
 F 2 "" H 3100 950 50  0000 C CNN
@@
 $EndComp
 $Comp
-L VCOM #PWR042
+L VCOM #PWR044
 U 1 1 5738A7C9
 P 3900 1600
-F 0 "#PWR042" H 3900 1450 50  0001 C CNN
+F 0 "#PWR044" H 3900 1450 50  0001 C CNN
 F 1 "VCOM" H 3900 1750 50  0000 C CNN
 F 2 "" H 3900 1600 50  0000 C CNN
@@
 $EndComp
 $Comp
-L GNDA #PWR043
+L GNDA #PWR045
 U 1 1 5738B8B9
 P 3600 1150
-F 0 "#PWR043" H 3600 900 50  0001 C CNN
+F 0 "#PWR045" H 3600 900 50  0001 C CNN
 F 1 "GNDA" H 3600 1000 50  0000 C CNN
 F 2 "" H 3600 1150 50  0000 C CNN
@@
 $EndComp
 Wire Wire Line
-	2450 3300 2750 3300
+	1600 3300 2750 3300
 Wire Wire Line
 	2600 3150 2600 3300
 Connection ~ 2600 3300
 Wire Wire Line
-	2450 3500 2750 3500
+	1600 3500 2750 3500
 Wire Wire Line
 	2600 3500 2600 3950
@@
 	2600 2850 2600 2750
 Wire Wire Line
-	2600 5000 2900 5000
+	1750 5000 2900 5000
 Wire Wire Line
 	2750 4850 2750 5000
 Connection ~ 2750 5000
 Wire Wire Line
-	2600 5200 2900 5200
+	1750 5200 2900 5200
 Wire Wire Line
 	2750 5200 2750 5650
@@
 	3900 5100 4050 5100
 Wire Wire Line
-	1850 5000 2300 5000
-Wire Wire Line
-	1850 5200 2300 5200
+	1000 5000 1450 5000
+Wire Wire Line
+	1000 5200 1450 5200
 Wire Wire Line
 	2750 4550 2750 4450
@@
 	1850 6600 2300 6600
 $Comp
-L VCOM #PWR044
+L VCOM #PWR046
 U 1 1 573B619B
 P 2250 6850
-F 0 "#PWR044" H 2250 6700 50  0001 C CNN
+F 0 "#PWR046" H 2250 6700 50  0001 C CNN
 F 1 "VCOM" H 2250 7000 50  0000 C CNN
 F 2 "" H 2250 6850 50  0000 C CNN
@@
 $EndComp
 Wire Wire Line
-	2150 3300 1850 3300
-Wire Wire Line
-	2150 3500 1850 3500
+	1300 3300 1000 3300
+Wire Wire Line
+	1300 3500 1000 3500
 Text Notes 3600 7400 2    60   ~ 0
 DO NOT OMIT
@@
 	2800 4150 2800 3950
 Connection ~ 2800 3950
-Text HLabel 1850 3300 0    60   Input ~ 0
-P_LEFT
-Text HLabel 1850 3500 0    60   Input ~ 0
-N_LEFT
-Text HLabel 1850 5000 0    60   Input ~ 0
-P_RIGHT
-Text HLabel 1850 5200 0    60   Input ~ 0
-N_RIGHT
+Text HLabel 1000 3300 0    60   Input ~ 0
+LO_P
+Text HLabel 1000 3500 0    60   Input ~ 0
+LO_N
+Text HLabel 1000 5000 0    60   Input ~ 0
+RO_P
+Text HLabel 1000 5200 0    60   Input ~ 0
+RO_N
 Text HLabel 4850 5100 2    60   Output ~ 0
 RIGHT_OUT
@@
 Text Label 1850 6600 2    60   ~ 0
 RIGHT_SE
+Text Label 2550 3300 2    60   ~ 0
+LEFT_OPAMP+
+Text Label 2550 3500 2    60   ~ 0
+LEFT_OPAMP-
+Text Label 2500 5000 2    60   ~ 0
+RIGHT_OPAMP+
+Text Label 2500 5200 2    60   ~ 0
+RIGHT_OPAMP-
+Text Label 1250 3300 2    60   ~ 0
+LO_P
+Text Label 1250 3500 2    60   ~ 0
+LO_N
+Text Label 1350 5200 2    60   ~ 0
+RO_N
+Text Label 1350 5000 2    60   ~ 0
+RO_P
 $EndSCHEMATC
