File: hardware/musamasiina.kicad_pcb (KiCad board)
At the start: 4 copper layers, 32.5 x 40 mm, 50 parts, among them P1 USB_OTG, P2 CONN_01X04, P3 CONN_02X03, P4 CONN_01X06, Q1 Q_NMOS_DGS, U1 WT32, U2 MIC5233-3.3, U3 LT6221, U4 TPS22860, U5 CD143A-SR05, U6 LM2776, U7 CD143A-SR05

Commit message: Finalize design
Parts:
- removed D1: D_Schottky, footprints:SOD323-M
- added C8: 2u2, footprints:SMD0402-CAP-N, F.Cu at (126.0, 63.2)
- added G***: LOGO, LOGO, B.Cu at (119.0, 77.0)
- U2: footprint footprints:SOT23-6-M -> footprints:SOT23-5-M
Connections:
- BT1 pad 2: GNDA -> GNDD
- C10 pad 1: +5V -> +BATT
- P4 pad 2: Net-(P4-Pad2) -> /CS
- U2 pad 1: +5V -> +BATT
Routing:
- net /CS: track 0.00 -> 41.4 mm, vias 0 -> 2
- net +5V: track 106.5 -> 92.6 mm
- net +BATT: track 64.1 -> 68.8 mm, vias 4 -> 3
- net /Power Supply/ENABLE: track 49.7 -> 51.9 mm, vias 2 -> 3
- net VDD: track 18.3 -> 19.9 mm
- net GNDA: track 20.6 -> 19.3 mm
- net VEE: track 21.5 -> 22.4 mm, vias 2 -> 3
- net GNDD: track 82.6 -> 83.4 mm
Other:
- board text added: "+5V"
- board text added: "CS"
- board text added: "GNDD"
- board text added: "Github/tkln"
- board text added: "Helsinki Hacklab"
- board text added: "MISO"
- board text added: "MOSI"
- board text added: "NC"
- board text added: "RESET"
- board text added: "RXD<-"
- board text added: "SCLK"
- board text added: "SPI"
- board text added: "Säätokerho"
- board text added: "TXD->"
- board text added: "UART"
